File: Circuit_layout/Circuit_layout.kicad_pcb (KiCad board)
At the start: 2 copper layers, 177.8 x 127 mm, 182 parts, among them CON1 AVR-JTAG-10, J1 Spare_Conns, J4 Motor_Ctrl, J5 RJ12, P1 TSV, P2 CONN_02X10, P3 CONN_02X07, Q1 ZVP4525G, Q2 MMBF170, Q3 MMBF170, SW1 SW_PUSH, SW2 TS5A3159-Q1, SW3 JS202011CQN, U1 RUW15SL12C, U10 MCP2551-I/SN, U11 TLP293, U12 TLP293, U13 PDQ10-D, U14 Mounting_hole, U15 Mounting_hole, U17 MCP6004, U18 TS912, U19 ACPL-C870, U2 MCP6002, U20 ACPL-C870, U21 MCP6001, U22 TS372, U23 TLP293, U24 TLP293, U25 Mounting_hole, U26 Mounting_hole, U27 TLP293, U3 MCP6004, U4 LM95071-Q1, U5 LM7810CT, U6 TS912, U7 AT90CAN128-A, U8 74ACT11030, U9 TLP293, Y1 10MHz

Commit message: Generated gerber and drill files for board ordering
Parts:
- removed +5DC/DC1: +5DC/DC, Measurement_Points:Measurement_Point_Round-SMD-Pad_Big
- removed P1: TSV, custom_footprints:AMPCONN_2
- removed P2: CONN_02X10, Connect:IDC_Header_Straight_20pins
- removed P3: CONN_02X07, Connect:IDC_Header_Straight_14pins
- removed R52: 250k, Resistors_SMD:R_0805_HandSoldering
- removed U24: TLP293, Housings_SSOP:SOP-4_4.4x2.8mm_Pitch1.27mm
- added D5: ~Throttle_PL, LEDs:LED_0805, F.Cu at (153.0, 94.2)
- added J10: Can_Iso, Connectors_Molex:Molex_MiniFit-JR-5556-04A_2x02x4.20mm_Straight, F.Cu at (156.2, 24.8)
- added J11: AIRs, Connectors_Molex:Molex_MiniFit-JR-5556-02A_2x01x4.20mm_Straight, F.Cu at (163.8, 24.8)
- added J12: IMD_Relay, Connectors_Molex:Molex_MiniFit-JR-5556-02A_2x01x4.20mm_Straight, F.Cu at (36.2, 99.1)
- added J13: TSV, custom_footprints:AMPCONN_2, F.Cu at (108.6, 142.2)
- added J2: Lights, Connectors_Molex:Molex_MiniFit-JR-5556-10A_2x05x4.20mm_Straight, F.Cu at (90.8, 24.8)
- added J3: Cockpit, Connectors_Molex:Molex_MiniFit-JR-5556-08A_2x04x4.20mm_Straight, F.Cu at (111.1, 24.8)
- added J6: Spare_Conns, custom_footprints:Molex_8x1_2.54mm, F.Cu at (83.8, 43.2)
- added J7: GLV_In, Connectors_Molex:Molex_MiniFit-JR-5556-06A_2x03x4.20mm_Straight, F.Cu at (127.6, 24.8)
- added J8: GLV_Out, Connectors_Molex:Molex_MiniFit-JR-5556-06A_2x03x4.20mm_Straight, F.Cu at (144.1, 24.8)
- added J9: IMD, custom_footprints:IMD_Header, F.Cu at (39.4, 67.3)
- added R47: 1k, Resistors_SMD:R_0805_HandSoldering, F.Cu at (142.9, 94.2)
- DC/DC_GND2: footprint Wire_Pads:SolderWirePad_single_2-5mmDrill -> Measurement_Points:Measurement_Point_Square-SMD-Pad_Big
- J1: value Spare_Conns -> Pedal_Cluster; footprint custom_footprints:Molex_8x1_2.54mm -> Connectors_Molex:Molex_MiniFit-JR-5556-12A_2x06x4.20mm_Straight
- R16: value 4.3K -> 250K
- R19: value 250k -> 4.3k
- Thrtl_LPF1, Thrtl_uC1: footprint Measurement_Points:Measurement_Point_Round-SMD-Pad_Big -> Measurement_Points:Measurement_Point_Square-SMD-Pad_Big
- moved HVPL_LV1 169.4 mm to (199.4, 73.2)
- moved R17 88.4 mm to (50.9, 51.6), turned to 180 degrees
- moved U10 78.1 mm to (148.0, 59.7)
- moved R37 78.1 mm to (155.6, 57.8)
- moved R44 78.1 mm to (155.6, 60.3)
- moved Q1 66.5 mm to (63.7, 41.9), turned to 0 degrees
- moved U27 32.1 mm to (130.2, 67.9), turned to 180 degrees
- moved Thrtl_uC1 28.5 mm to (97.0, 86.9)
- moved J1 26.1 mm to (66.0, 24.8), turned to 180 degrees
- moved APPS_DIFF1 25.3 mm to (79.5, 77.0)
- moved R27 16.1 mm to (138.6, 67.8), turned to 0 degrees
- moved C37 14.4 mm to (155.6, 62.9), turned to 180 degrees
- moved C6 9.79 mm to (128.8, 100.1)
- moved Y1 9.72 mm to (130.0, 103.1)
- moved C5 9.72 mm to (135.1, 101.9)
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Connections:
- net /CC_LED_CTRL renamed /SPARE_LED_CTRL
- J1 pad 1: UART_RX -> +24V
- J1 pad 2: UART_TX -> +24V
- J1 pad 3: SCL -> BP
- J1 pad 4: SDA -> Net-(J1-Pad4)
- J1 pad 5: Spare_OC -> APPS1_10
- J1 pad 6: Spare_ICP -> APPS1
- J1 pad 7: Spare_ADC_1 -> APPS1_RTN
- J1 pad 8: Spare_ADC_2 -> APPS2_5
- U27 pad 3: CC_LED -> SPARE_LED
- U7 pad 8: /BOT_uC -> Net-(U7-Pad8)
Routing:
- net HVPL: track 13.3 -> 266.9 mm
- net IMD_PWM: track 67.9 -> 233.7 mm
- net APPS2_5: track 7.62 -> 106.2 mm, vias 0 -> 3
- net APPS1_RTN: track 7.73 -> 102.4 mm, vias 0 -> 3
- net +24V_RTN: track 47.9 -> 123.3 mm, vias 0 -> 2
- net SPARE_LED: track 0.00 -> 74.7 mm, vias 0 -> 3
- net CH_GND: track 264.0 -> 196.8 mm, vias 31 -> 24
- net /BOT_uC: track 63.5 -> 0.00 mm, vias 4 -> 0
- net APPS1_10: track 159.9 -> 208.8 mm, vias 13 -> 15
- net Drive_BTN: track 45.7 -> 93.4 mm, vias 2 -> 3
- net /Throttle_PL: track 92.0 -> 139.0 mm, vias 4 -> 7
- net BP: track 41.6 -> 85.8 mm, vias 1 -> 4
- net BOT: track 42.7 -> 0.00 mm, vias 1 -> 0
- net SCL: track 144.5 -> 102.3 mm, vias 3 -> 6
- net APPS2: track 102.7 -> 144.3 mm, vias 2 -> 3
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Other:
- board size 177.8 x 127 mm -> 177.8 x 142.2 mm
- net class TSAL: clearance 0.254 -> 0.2032
- board text added: "Designed by: Peter Phelan"
- board text added: "~THRTL_PL"
- board text removed: "Designed by: Jack Plumb and Adam Ness"
