File: Circuit_layout/_saved_Circuit_layout.sch (KiCad schematic (older format))
At the start: 34 parts, among them Q3 MMBF170, SW1 SW_PUSH, SW3 JS202011CQN, U17 MCP6004, U4 LM95071-Q1, U7 AT90CAN128-A, U9 TLP293, Y1 10MHz

Commit message: Generated gerber and drill files for board ordering
Connections:
- net BOT_uC: no longer U7.8 (PE6(T3/INT6))
- no-connect marks 20 -> 21
Changed lines of the file:
@@
 Text Label 11100 6250 0    60   ~ 0
-BOT_uC
-Text Label 6600 5100 0    60   ~ 0
 BOT_uC
 $Comp
@@
 Text Notes 3800 2950 0    99   ~ 0
 Temp. Sensor
-Wire Wire Line
-	7200 5100 6600 5100
 NoConn ~ 9800 3600
 Wire Wire Line
@@
 Wire Wire Line
 	9800 2000 9850 2000
+NoConn ~ 7200 5100
 $EndSCHEMATC
