File: Circuit_layout/_saved_StatusLights.sch (KiCad schematic (older format))
At the start: 24 parts, among them Q1 ZVP4525G, U1 RUW15SL12C, U11 TLP293, U12 TLP293, U27 TLP293

Commit message: Generated gerber and drill files for board ordering
Parts:
- C3: footprint Capacitors_THT:CP_Radial_D10.0mm_P5.00mm -> Capacitors_SMD:CP_Elec_8x10
Changed lines of the file:
@@
 F 0 "C3" H 1225 5700 50  0000 L CNN
 F 1 "10uF" H 1225 5500 50  0000 L CNN
-F 2 "Capacitors_THT:CP_Radial_D10.0mm_P5.00mm" H 1238 5450 50  0001 C CNN
+F 2 "Capacitors_SMD:CP_Elec_8x10" H 1238 5450 50  0001 C CNN
 F 3 "" H 1200 5600 50  0000 C CNN
 F 4 "490-3550-1-ND" H 1200 5600 60  0001 C CNN "DigiKey P/N"
