File: Circuit_layout/_saved_ThrottlePlausibility.sch (KiCad schematic (older format))
At the start: 69 parts, among them Q2 MMBF170, SW2 TS5A3159-Q1, U18 TS912, U2 MCP6002, U22 TS372, U23 TLP293, U24 TLP293, U3 MCP6004, U5 LM7810CT, U6 TS912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

Commit message: Generated gerber and drill files for board ordering
Parts:
- removed R52: 250k, Resistors_SMD:R_0805_HandSoldering, symbol R
- removed U24: TLP293, Housings_SSOP:SOP-4_4.4x2.8mm_Pitch1.27mm, symbol TLP291
- added D5: ~Throttle_PL, LEDs:LED_0805, symbol LED_ALT
- added R47: 1k, Resistors_SMD:R_0805_HandSoldering, symbol R
Connections:
- net GND: now also D5.1 (K)
- net Throttle_PL: now also R47.2
- new net: D5.2 (A), R47.1
Other:
- note added: "RED"
- note removed: "Brake Overtravel"
Changed lines of the file:
@@
 Text GLabel 3250 850  0    60   Input ~ 0
 APPS1_RTN
-Text Label 13500 2450 0    60   ~ 0
-RTN_GLV
-Text Notes 13450 1900 0    99   ~ 0
-Brake Overtravel
-Text Label 3450 1500 0    60   ~ 0
-BOT
-Text GLabel 3250 1500 0    60   Input ~ 0
-BOT
 Text HLabel 3200 1950 0    60   Input ~ 0
 BOT_uC
@@
 BOT_uC
 $Comp
-L TLP291 U24
-U 1 1 58BF52E8
-P 14550 2350
-F 0 "U24" H 14350 2550 50  0000 L CNN
-F 1 "TLP293" H 14550 2550 50  0000 L CNN
-F 2 "Housings_SSOP:SOP-4_4.4x2.8mm_Pitch1.27mm" H 14350 2150 50  0001 L CIN
-F 3 "" H 14550 2350 50  0000 L CNN
-F 4 "TLP293(GB-TPLECT-ND" H 14550 2350 60  0001 C CNN "DigiKey P/N"
-F 5 "http://www.digikey.com/product-detail/en/toshiba-semiconductor-and-storage/TLP293(GB-TPL,E/TLP293(GB-TPLECT-ND/4562965" H 14550 2350 60  0001 C CNN "URL"
-F 6 "TLP293(GB-TPLE" H 14550 2350 60  0001 C CNN "Man P/N"
-F 7 "http://www.digikey.com/product-detail/en/toshiba-semiconductor-and-storage/TLP291(GB-TP,SE/TLP291(GB-TPSECT-ND/4562949" H 14550 2350 60  0001 C CNN "TLP291"
-	1    14550 2350
-	1    0    0    -1
-$EndComp
-$Comp
 L GND #PWR095
-U 1 1 58BF5303
-P 14950 2550
-F 0 "#PWR095" H 14950 2300 50  0001 C CNN
-F 1 "GND" H 14950 2400 50  0000 C CNN
-F 2 "" H 14950 2550 50  0000 C CNN
-F 3 "" H 14950 2550 50  0000 C CNN
-	1    14950 2550
-	1    0    0    -1
-$EndComp
-Text Label 14950 2250 0    60   ~ 0
-BOT_uC
-Text Label 13500 2250 0    60   ~ 0
-BOT
-$Comp
-L GND #PWR096
 U 1 1 58C17F0F
 P 3800 9450
-F 0 "#PWR096" H 3800 9200 50  0001 C CNN
+F 0 "#PWR095" H 3800 9200 50  0001 C CNN
 F 1 "GND" H 3800 9300 50  0000 C CNN
 F 2 "" H 3800 9450 50  0000 C CNN
@@
 APPS_10
 $Comp
-L GND #PWR097
+L GND #PWR096
 U 1 1 58BFE2A1
 P 2550 9450
-F 0 "#PWR097" H 2550 9200 50  0001 C CNN
+F 0 "#PWR096" H 2550 9200 50  0001 C CNN
 F 1 "GND" H 2550 9300 50  0000 C CNN
 F 2 "" H 2550 9450 50  0000 C CNN
@@
 $EndComp
 $Comp
-L GND #PWR098
+L GND #PWR097
 U 1 1 58BFFFDF
 P 2000 9450
-F 0 "#PWR098" H 2000 9200 50  0001 C CNN
+F 0 "#PWR097" H 2000 9200 50  0001 C CNN
 F 1 "GND" H 2000 9300 50  0000 C CNN
 F 2 "" H 2000 9450 50  0000 C CNN
@@
 $EndComp
 $Comp
-L GND #PWR099
+L GND #PWR098
 U 1 1 58C09A9E
 P 5150 9450
-F 0 "#PWR099" H 5150 9200 50  0001 C CNN
+F 0 "#PWR098" H 5150 9200 50  0001 C CNN
 F 1 "GND" H 5150 9300 50  0000 C CNN
 F 2 "" H 5150 9450 50  0000 C CNN
@@
 $EndComp
 $Comp
-L GND #PWR0100
+L GND #PWR099
 U 1 1 58C09EB8
 P 4600 9450
-F 0 "#PWR0100" H 4600 9200 50  0001 C CNN
+F 0 "#PWR099" H 4600 9200 50  0001 C CNN
 F 1 "GND" H 4600 9300 50  0000 C CNN
 F 2 "" H 4600 9450 50  0000 C CNN
@@
 $EndComp
 $Comp
-L +24V #PWR0101
+L +24V #PWR0100
 U 1 1 58C0FB3A
 P 1350 3950
-F 0 "#PWR0101" H 1350 3800 50  0001 C CNN
+F 0 "#PWR0100" H 1350 3800 50  0001 C CNN
 F 1 "+24V" H 1350 4090 50  0000 C CNN
 F 2 "" H 1350 3950 50  0000 C CNN
@@
 APPS_10
 $Comp
-L GND #PWR0102
+L GND #PWR0101
 U 1 1 58C13EC3
 P 5400 6550
-F 0 "#PWR0102" H 5400 6300 50  0001 C CNN
+F 0 "#PWR0101" H 5400 6300 50  0001 C CNN
 F 1 "GND" H 5400 6400 50  0000 C CNN
 F 2 "" H 5400 6550 50  0000 C CNN
@@
 Connection ~ 1450 4050
 Wire Wire Line
-	3250 1500 3450 1500
-Wire Wire Line
 	3200 1950 3400 1950
-Wire Wire Line
-	13500 2250 13800 2250
-Wire Wire Line
-	14100 2250 14250 2250
-Wire Wire Line
-	13500 2450 14250 2450
 Wire Notes Line
 	1150 9050 1150 8750
@@
 	3800 8150 3800 7950
 Wire Wire Line
-	14850 2450 14950 2450
-Wire Wire Line
-	14950 2450 14950 2550
-Wire Wire Line
-	14850 2250 14950 2250
-Wire Wire Line
 	2550 9300 2550 9450
 Wire Wire Line
@@
 APPS1_b
 $Comp
-L GND #PWR0103
+L GND #PWR0102
 U 1 1 58C2062A
 P 2700 6250
-F 0 "#PWR0103" H 2700 6000 50  0001 C CNN
+F 0 "#PWR0102" H 2700 6000 50  0001 C CNN
 F 1 "GND" H 2700 6100 50  0000 C CNN
 F 2 "" H 2700 6250 50  0000 C CNN
@@
 $EndComp
 $Comp
-L GND #PWR0104
+L GND #PWR0103
 U 1 1 58C20630
 P 2200 6550
-F 0 "#PWR0104" H 2200 6300 50  0001 C CNN
+F 0 "#PWR0103" H 2200 6300 50  0001 C CNN
 F 1 "GND" H 2200 6400 50  0000 C CNN
 F 2 "" H 2200 6550 50  0000 C CNN
@@
 $EndComp
 $Comp
-L +5V #PWR0105
+L +5V #PWR0104
 U 1 1 58C2185C
 P 1150 5950
-F 0 "#PWR0105" H 1150 5800 50  0001 C CNN
+F 0 "#PWR0104" H 1150 5800 50  0001 C CNN
 F 1 "+5V" H 1150 6090 50  0000 C CNN
 F 2 "" H 1150 5950 50  0000 C CNN
@@
 $EndComp
 $Comp
-L GND #PWR0106
+L GND #PWR0105
 U 1 1 58C331D8
 P 12800 2550
-F 0 "#PWR0106" H 12800 2300 50  0001 C CNN
+F 0 "#PWR0105" H 12800 2300 50  0001 C CNN
 F 1 "GND" H 12800 2400 50  0000 C CNN
 F 2 "" H 12800 2550 50  0000 C CNN
@@
 Wire Wire Line
 	12700 2250 12800 2250
-$Comp
-L R R52
-U 1 1 58C344AC
-P 13950 2250
-F 0 "R52" V 14030 2250 50  0000 C CNN
-F 1 "250k" V 13950 2250 50  0000 C CNN
-F 2 "Resistors_SMD:R_0805_HandSoldering" V 13880 2250 50  0001 C CNN
-F 3 "" H 13950 2250 50  0000 C CNN
-F 4 "P249KCCT-ND" V 13950 2250 60  0001 C CNN "DigiKey P/N"
-F 5 "http://www.digikey.com/product-detail/en/panasonic-electronic-components/ERJ-6ENF2493V/P249KCCT-ND/119664" V 13950 2250 60  0001 C CNN "URL"
-F 6 "ERJ-6ENF2493V" V 13950 2250 60  0001 C CNN "Man P/N"
-F 7 "RES SMD 249K OHM 1% 1/8W 0805" V 13950 2250 60  0001 C CNN "Description"
-F 8 "0.10" V 13950 2250 60  0001 C CNN "Cost"
-	1    13950 2250
-	0    -1   -1   0
-$EndComp
 Text Notes 1200 7650 0    99   ~ 0
 APPS 5V Offset Bias
@@
 Connection ~ 10150 4900
 $Comp
-L +5V #PWR0107
+L +5V #PWR0106
 U 1 1 58C55D3B
 P 10150 4800
-F 0 "#PWR0107" H 10150 4650 50  0001 C CNN
+F 0 "#PWR0106" H 10150 4650 50  0001 C CNN
 F 1 "+5V" H 10150 4940 50  0000 C CNN
 F 2 "" H 10150 4800 50  0000 C CNN
@@
 $EndComp
 $Comp
-L GND #PWR0108
+L GND #PWR0107
 U 1 1 58C5A996
 P 13850 5700
-F 0 "#PWR0108" H 13850 5450 50  0001 C CNN
+F 0 "#PWR0107" H 13850 5450 50  0001 C CNN
 F 1 "GND" H 13850 5550 50  0000 C CNN
 F 2 "" H 13850 5700 50  0000 C CNN
@@
 $EndComp
 $Comp
-L +5V #PWR0109
+L +5V #PWR0108
 U 1 1 58D04CF9
 P 15050 5200
-F 0 "#PWR0109" H 15050 5050 50  0001 C CNN
+F 0 "#PWR0108" H 15050 5050 50  0001 C CNN
 F 1 "+5V" H 15050 5340 50  0000 C CNN
 F 2 "" H 15050 5200 50  0000 C CNN
@@
 Look at datasheet for \nfootprint design specs
 $Comp
-L GND #PWR0110
+L GND #PWR0109
 U 1 1 58D1EB87
 P 10650 5550
-F 0 "#PWR0110" H 10650 5300 50  0001 C CNN
+F 0 "#PWR0109" H 10650 5300 50  0001 C CNN
 F 1 "GND" H 10650 5400 50  0000 C CNN
 F 2 "" H 10650 5550 50  0000 C CNN
@@
 	10650 5550 10650 5450
 $Comp
-L +5V #PWR0111
+L +5V #PWR0110
 U 1 1 58D1EDC9
 P 10650 4950
-F 0 "#PWR0111" H 10650 4800 50  0001 C CNN
+F 0 "#PWR0110" H 10650 4800 50  0001 C CNN
 F 1 "+5V" H 10650 5090 50  0000 C CNN
 F 2 "" H 10650 4950 50  0000 C CNN
@@
 $EndComp
 $Comp
-L +5V #PWR0112
+L +5V #PWR0111
 U 1 1 5A7D5A7D
 P 12600 5900
-F 0 "#PWR0112" H 12600 5750 50  0001 C CNN
+F 0 "#PWR0111" H 12600 5750 50  0001 C CNN
 F 1 "+5V" H 12600 6040 50  0000 C CNN
 F 2 "" H 12600 5900 50  0000 C CNN
@@
 $EndComp
 $Comp
-L GND #PWR0113
+L GND #PWR0112
 U 1 1 5A7D5B54
 P 12600 6900
-F 0 "#PWR0113" H 12600 6650 50  0001 C CNN
+F 0 "#PWR0112" H 12600 6650 50  0001 C CNN
 F 1 "GND" H 12600 6750 50  0000 C CNN
 F 2 "" H 12600 6900 50  0000 C CNN
@@
 $EndComp
 $Comp
-L GND #PWR0114
+L GND #PWR0113
 U 1 1 5A846229
 P 12000 7100
-F 0 "#PWR0114" H 12000 6850 50  0001 C CNN
+F 0 "#PWR0113" H 12000 6850 50  0001 C CNN
 F 1 "GND" H 12000 6950 50  0000 C CNN
 F 2 "" H 12000 7100 50  0000 C CNN
@@
 Connection ~ 11400 6600
 Connection ~ 13350 6500
+$Comp
+L R R47
+U 1 1 5A92FC89
+P 11250 8100
+F 0 "R47" V 11330 8100 50  0000 C CNN
+F 1 "1k" V 11250 8100 50  0000 C CNN
+F 2 "Resistors_SMD:R_0805_HandSoldering" V 11180 8100 50  0001 C CNN
+F 3 "" H 11250 8100 50  0000 C CNN
+F 4 "P249KCCT-ND" V 11250 8100 60  0001 C CNN "DigiKey P/N"
+F 5 "http://www.digikey.com/product-detail/en/panasonic-electronic-components/ERJ-6ENF2493V/P249KCCT-ND/119664" V 11250 8100 60  0001 C CNN "URL"
+F 6 "ERJ-6ENF2493V" V 11250 8100 60  0001 C CNN "Man P/N"
+F 7 "RES SMD 249K OHM 1% 1/8W 0805" V 11250 8100 60  0001 C CNN "Description"
+F 8 "0.10" V 11250 8100 60  0001 C CNN "Cost"
+	1    11250 8100
+	0    1    1    0
+$EndComp
+$Comp
+L LED_ALT D5
+U 1 1 5A9328C2
+P 11750 8100
+F 0 "D5" H 11750 8200 50  0000 C CNN
+F 1 "~Throttle_PL" H 11750 7950 50  0000 C CNN
+F 2 "LEDs:LED_0805" H 11750 8100 50  0001 C CNN
+F 3 "" H 11750 8100 50  0001 C CNN
+	1    11750 8100
+	-1   0    0    1
+$EndComp
+$Comp
+L GND #PWR0114
+U 1 1 5A934199
+P 12000 8200
+F 0 "#PWR0114" H 12000 7950 50  0001 C CNN
+F 1 "GND" H 12000 8050 50  0000 C CNN
+F 2 "" H 12000 8200 50  0000 C CNN
+F 3 "" H 12000 8200 50  0000 C CNN
+	1    12000 8200
+	1    0    0    -1
+$EndComp
+Wire Wire Line
+	11400 8100 11600 8100
+Wire Wire Line
+	11900 8100 12000 8100
+Wire Wire Line
+	12000 8100 12000 8200
+Text Label 10550 8100 0    60   ~ 0
+Throttle_PL
+Wire Wire Line
+	10550 8100 11100 8100
+Text Notes 11650 8350 0    60   ~ 0
+RED
 $EndSCHEMATC
