File: Circuit_layout/Can_tcvr.sch (KiCad schematic (older format))
At the start: 4 parts, among them U10 MCP2551-I/SN

Commit message: Completed errata changes
Committing before annotation, footprint assignment, and board relayout for backup purposes
Parts:
- U10: symbol MCP2551-I/SN -> MCP2551-I/SN-RESCUE-Circuit_layout
Changed lines of the file:
@@
 EESchema Schematic File Version 2
 LIBS:Circuit_layout-rescue
-LIBS:TSI_KiCad_Lib
 LIBS:TSI_HV_Isolater-cache
 LIBS:74xgxx
@@
 LIBS:xilinx
 LIBS:Zilog
-LIBS:pacman-main-cache
 LIBS:bss84
 LIBS:+10v
@@
 $EndDescr
 $Comp
-L MCP2551-I/SN U10
+L MCP2551-I/SN-RESCUE-Circuit_layout U10
 U 1 1 58A630DD
 P 3800 1500
