File: Circuit_layout/isolators.sch (KiCad schematic (older format))
At the start: 35 parts, among them U17 MCP6004, U19 ACPL-C870, U20 ACPL-C870, U21 MCP6001

Commit message: Completed errata changes
Committing before annotation, footprint assignment, and board relayout for backup purposes
Parts:
- R58: value 24.9k -> 15k
- U21: symbol MCP6001 -> MCP6001-RESCUE-Circuit_layout
Other:
- note removed: "Current R58 (24.9k) results in incorrect amplification.\nReplaced w/ 15k"
Changed lines of the file:
@@
 EESchema Schematic File Version 2
 LIBS:Circuit_layout-rescue
-LIBS:TSI_KiCad_Lib
 LIBS:TSI_HV_Isolater-cache
 LIBS:74xgxx
@@
 LIBS:xilinx
 LIBS:Zilog
-LIBS:pacman-main-cache
 LIBS:bss84
 LIBS:+10v
@@
 I/O_Ground
 $Comp
-L MCP6001 U21
+L MCP6001-RESCUE-Circuit_layout U21
 U 1 1 58B7DBA9
 P 7950 2700
@@
 P 3700 2600
 F 0 "R58" V 3780 2600 50  0000 C CNN
-F 1 "24.9k" V 3700 2600 50  0000 C CNN
+F 1 "15k" V 3700 2600 50  0000 C CNN
 F 2 "Resistors_SMD:R_0805_HandSoldering" V 3630 2600 50  0001 C CNN
 F 3 "" H 3700 2600 50  0000 C CNN
@@
 	3350 4100 3900 4100
 Connection ~ 3550 4100
-Text Notes 2800 2400 0    39   ~ 0
-Current R58 (24.9k) results in incorrect amplification.\nReplaced w/ 15k
 $EndSCHEMATC

Commit message: Backup before pcb relayout
Parts:
- +5HV1: footprint Measurement_Points:Measurement_Point_Round-SMD-Pad_Big -> custom_footprints:TSSOP-16-1EP_4.4x5mm_Pitch0.65mm
Changed lines of the file:
@@
 F 0 "+5HV1" H 9500 2670 50  0000 C CNN
 F 1 "+5HV" H 9500 2600 50  0000 C CNN
-F 2 "Measurement_Points:Measurement_Point_Round-SMD-Pad_Big" H 9700 2400 50  0001 C CNN
+F 2 "custom_footprints:TSSOP-16-1EP_4.4x5mm_Pitch0.65mm" H 9700 2400 50  0001 C CNN
 F 3 "" H 9700 2400 50  0000 C CNN
 	1    9500 2400
